Commit message: add part3 MATLAB script for plotting data

File: rbebot_description/urdf/rbebot.urdf (robot description, URDF)
Before this commit: robot rbebot, 8 links, 7 joints
Joints:
- joint joint1: limit effort=100.0 velocity=0.1 -> effort=1000.0 velocity=1.0
- joint joint2: limit lower=-2.09 upper=2.09 effort=1000.0 velocity=0.5 -> lower=-2.09 upper=2.09 effort=1000.0 velocity=1.0
- joint joint3: limit lower=-0.35 upper=0.35 effort=100.0 velocity=0.5 -> lower=-0.35 upper=0.35 effort=1000.0 velocity=0.5
